Commit message: Set provisional joint limits and update limit notes
Co-Authored-By: Claude Opus 5.5 <noreply@anthropic.com>

File: src/arctos_description/urdf/arctos.urdf (robot description, URDF)
Before this commit: robot arctos, 7 links, 6 joints
Joints:
- joint joint_1: limit lower=0 upper=0 effort=0 velocity=0 -> lower=-1.570796 upper=1.570796 effort=0 velocity=0
- joint joint_2: limit lower=0 upper=0 effort=0 velocity=0 -> lower=-1.256637 upper=2.094395 effort=0 velocity=0
- joint joint_3: limit lower=0 upper=0 effort=0 velocity=0 -> lower=-1.570796 upper=1.029744 effort=0 velocity=0
- joint joint_4: limit lower=0 upper=0 effort=0 velocity=0 -> lower=-1.570796 upper=1.570796 effort=0 velocity=0
- joint joint_5: limit lower=0 upper=0 effort=0 velocity=0 -> lower=-1.570796 upper=1.570796 effort=0 velocity=0
- joint joint_6: limit lower=0 upper=0 effort=0 velocity=0 -> lower=-1.570796 upper=1.570796 effort=0 velocity=0

Commit message: Compute joint limits from CAD collisions and add tool frames
Add joint_limits.py to sweep each joint over the link meshes and set
limits at the nearest collision angle divided by 1.5. Apply the results
to the URDF, add ROS-Industrial flange and tool0 frames, document the
rule, and require step-by-step work on the user's command.

Co-Authored-By: Claude Opus 5.5 <noreply@anthropic.com>

File: src/arctos_description/urdf/arctos.urdf (robot description, URDF)
Before this commit: robot arctos, 7 links, 6 joints
Links:
- added link flange
- added link tool0
Joints:
- added joint flange-tool0: type fixed, parent flange, child tool0, origin xyz=0 0 0 rpy=3.141593 -1.570796 0
- added joint joint_6-flange: type fixed, parent tool_link, child flange, origin xyz=0.013 0 0 rpy=0 0 0
- joint joint_1: limit lower=-1.570796 upper=1.570796 effort=0 velocity=0 -> lower=-3.141593 upper=3.141593 effort=0 velocity=0
- joint joint_2: limit lower=-1.256637 upper=2.094395 effort=0 velocity=0 -> lower=-0.933024 upper=0.883573 effort=0 velocity=0
- joint joint_3: limit lower=-1.570796 upper=1.029744 effort=0 velocity=0 -> lower=-2.370012 upper=0.802851 effort=0 velocity=0
- joint joint_4: limit lower=-1.570796 upper=1.570796 effort=0 velocity=0 -> lower=-3.141593 upper=3.141593 effort=0 velocity=0
- joint joint_5: limit lower=-1.570796 upper=1.570796 effort=0 velocity=0 -> lower=-3.141593 upper=3.141593 effort=0 velocity=0
- joint joint_6: limit lower=-1.570796 upper=1.570796 effort=0 velocity=0 -> lower=-3.141593 upper=3.141593 effort=0 velocity=0

Commit message: Sync working-copy collision meshes, docs, and collision demo
Baseline copy of uncommitted main-checkout changes (result.json excluded).

Co-Authored-By: Claude Opus 5.5 <noreply@anthropic.com>

File: src/arctos_description/urdf/arctos.urdf (robot description, URDF)
Before this commit: robot arctos, 9 links, 8 joints
Links:
- link base_link: geometry collision mesh filename=package://arctos_description/meshes/collision/base_link.stl scale=0.001 0.001 0.001; visual mesh filename=package://arctos_description/meshes/base_link.stl scale=0.001 0.001 0.001
- link elbow_link: geometry collision mesh filename=package://arctos_description/meshes/collision/elbow_link.stl scale=0.001 0.001 0.001; visual mesh filename=package://arctos_description/meshes/elbow_link.stl scale=0.001 0.001 0.001
- link shoulder_link: geometry collision mesh filename=package://arctos_description/meshes/collision/shoulder_link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 scale=0.001 0.001 0.001; visual mesh filename=package://arctos_description/meshes/shoulder_link.stl scale=0.001 0.001 0.001
- link tool_link: geometry collision mesh filename=package://arctos_description/meshes/collision/tool_link.stl scale=0.001 0.001 0.001; visual mesh filename=package://arctos_description/meshes/tool_link.stl scale=0.001 0.001 0.001
- link upper_arm_link: geometry collision mesh filename=package://arctos_description/meshes/collision/upper_arm_lin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 scale=0.001 0.001 0.001; visual mesh filename=package://arctos_description/meshes/upper_arm_link.stl scale=0.001 0.001 0.001
- link wrist_pitch_link: geometry collision mesh filename=package://arctos_description/meshes/collision/wrist_pitch_l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 scale=0.001 0.001 0.001; visual mesh filename=package://arctos_description/meshes/wrist_pitch_link.stl scale=0.001 0.001 0.001
- link wrist_roll_link: geometry collision mesh filename=package://arctos_description/meshes/collision/wrist_roll_li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 scale=0.001 0.001 0.001; visual mesh filename=package://arctos_description/meshes/wrist_roll_link.stl scale=0.001 0.001 0.001
